Commit message: wheels placed right spot | one wheel little misplaced

File: urdf/hola_bot.urdf (robot description, URDF)
Before this commit: robot hola_bot, 2 links, 1 joints
Links:
- added link left_wheel, mass 0.062; collision cylinder length=0.02 radius=.03; visual mesh filename=package://task1/meshes/wheel.STL
- added link right_wheel, mass 0.062; collision cylinder length=0.02 radius=.03; visual mesh filename=package://task1/meshes/wheel.STL
Joints:
- added joint left_joint: type continuous, parent base_link, child left_wheel, origin xyz=-0.15154 -0.087275  -0.0335 rpy=0 0 2.0944, axis 0 -1 0, limit effort=5 velocity=5
- added joint right_joint: type continuous, parent base_link, child right_wheel, origin xyz=0.15154 -0.087275  -0.0335 rpy=0 0 1.0472, axis 0 -1 0, limit effort=5 velocity=5
